File: uaefi.kicad_sch (KiCad schematic)
At the start: 71 parts, among them J1 Conn_02x02_Odd_Even, J1 USB_B_Mini, J1 USB_C, J10 5569-16A2, J11 Conn_02x02_Odd_Even, J12 Conn_02x02_Odd_Even, J13 Conn_02x02_Odd_Even, J14 Conn_02x02_Odd_Even, J15 Conn_02x02_Odd_Even, J16 Conn_02x02_Odd_Even, J17 Conn_01x06, J17 Conn_02x02_Odd_Even, J18 Conn_02x02_Odd_Even, J19 Conn_02x02_Odd_Even, J2 5569-20A2, J20 Conn_02x02_Odd_Even, J21 Conn_02x02_Odd_Even, J22 Conn_02x02_Odd_Even, J24 Conn_02x02_Odd_Even, J3 5569-06A2, J4 5569-08A2, J5 5569-18A2, J5 Conn_01x05_Male, M1 Module-power_12and5V-0.3, M3 Module-knock-0.2, M3 Module-vr-discrete-0.5, M4 Module-vr-max9924-0.1, M5 Module-wbo-0.6, M6 Module:mega-mcu100/0.3, M7 Module-can-0.1, P1 Pad, P2 Pad, P3 Pad, P4 Pad, P5 Pad, P6 Pad, P7 Pad, P8 Pad, U4 JDY-33

Commit message: uaefi-moto schematic: 2x Superseal 34, 4x EGT, second WBO, no DC drivers [skip ci]
- J2/J3/J4/J5/J10 Mini-Fit replaced by J30 (TE 6437288-1) and J31 (TE 6437288-2)
- three more EGT sheet instances (CS on DC1_PWM/DC1_DIR/DC2_PWM) + four PCC-SMP-K sockets
- second Module-wbo-0.6 (M8) strapped to hardware index 5
- DC Driver sheets and their fuses F3/F4 removed
- PTC F11 for +12V hall supply
- ERC: 0 errors; netlist verified against original

Co-Authored-By: Claude Opus 5.5 <noreply@anthropic.com>
Parts:
- removed F3, F4: Fuse, Fuse:Fuse_1206_3216Metric_Pad1.42x1.75mm_HandSolder, symbol Device:Fuse
- removed J10: 5569-16A2, Connector_Molex:Molex_Mini-Fit_Jr_5569-16A2_2x08_P4.20mm_Horizontal, symbol Connector_Generic:Conn_02x08_Top_Bottom
- removed J2: 5569-20A2, Connector_Molex:Molex_Mini-Fit_Jr_5569-20A2_2x10_P4.20mm_Horizontal, symbol Connector_Generic:Conn_02x10_Top_Bottom
- removed J3: 5569-06A2, Connector_Molex:Molex_Mini-Fit_Jr_5569-06A2_2x03_P4.20mm_Horizontal, symbol Connector_Generic:Conn_02x03_Top_Bottom
- removed J4: 5569-08A2, Connector_Molex:Molex_Mini-Fit_Jr_5569-08A2_2x04_P4.20mm_Horizontal, symbol Connector_Generic:Conn_02x04_Top_Bottom
- removed J5: 5569-18A2, Connector_Molex:Molex_Mini-Fit_Jr_5569-18A2_2x09_P4.20mm_Horizontal, symbol Connector_Generic:Conn_02x09_Top_Bottom
- added F11: PTC 200mA hold, Fuse:Fuse_1206_3216Metric_Pad1.42x1.75mm_HandSolder, symbol Device:Fuse
- added J30: TE 6437288-1 (A, keying 1), Connectors:6437288-2, symbol Connectors:TE_6437288-2_34p
- added J31: TE 6437288-2 (B, keying 2), Connectors:6437288-2, symbol Connectors:TE_6437288-2_34p
- added J32: EGT1 PCC-SMP-K, moto:Omega_PCC-SMP-K, symbol Connector_Generic:Conn_01x02
- added J33: EGT2 PCC-SMP-K, moto:Omega_PCC-SMP-K, symbol Connector_Generic:Conn_01x02
- added J34: EGT3 PCC-SMP-K, moto:Omega_PCC-SMP-K, symbol Connector_Generic:Conn_01x02
- added J35: EGT4 PCC-SMP-K, moto:Omega_PCC-SMP-K, symbol Connector_Generic:Conn_01x02
- added M8: Module-wbo-0.6, hellen-one-wbo-0.6:wbo, symbol hellen-one-wbo-0.6:Module-wbo-0.6
Connections:
- net +12V: now also J30.1
- net +12V_RAW: now also F11.1, J30.25, J30.27
- net +5VA: now also M8.W1 (V5_IN)
- net +5VP: now also J31.1, J31.2
- net 12V_KEY: now also J30.2
- net 1_WBO_Ip: now also J31.27
- net 2_WBO_Vm: now also J31.28
- net 3_WBO_Heater: now also J30.26
- net 5_WBO_Rtrim: now also J31.30
- net 6_WBO_Un: now also J31.29
- net CAN+: now also J30.33, M8.W4 (CANH)
- net CAN-: now also J30.34, M8.W3 (CANL)
- net EGT+: now also J32.1 (Pin_1)
- net EGT-: now also J32.2 (Pin_2)
- net GND: now also J30.3, J30.32, J30.4, J30.5, J31.25, M8.G (GND)
- net GNDA: now also J31.3, J31.4, J31.5
- net IN_AUX1: now also J31.11
- net IN_AUX2: now also J31.12
- net IN_AUX3: now also J31.15
- net IN_BUTTON1: now also J31.20
- net IN_CLT: now also J31.8
- net IN_FLEX: now also J31.19
- net IN_HALL1: now also J31.16
- net IN_HALL2: now also J31.17
- net IN_HALL3: now also J31.18
- net IN_IAT: now also J31.9
- net IN_KNOCK_RAW: now also J31.26
- net IN_MAP: now also J31.10
- net IN_PPS1: now also J31.13
- net IN_PPS2: now also J31.14
- net IN_TPS1: now also J31.6
- net IN_TPS2: now also J31.7
- net OUT_IGN1: now also J30.13
- net OUT_IGN2: now also J30.14
- net OUT_IGN3: now also J30.15
- net OUT_IGN4: now also J30.16
- net OUT_IGN5: now also J30.17
- net OUT_IGN6: now also J30.18
- net OUT_INJ1: now also J30.7
- net OUT_INJ2: now also J30.8
- net OUT_INJ3: now also J30.9
- net OUT_INJ4: now also J30.10
- net OUT_INJ5: now also J30.11
- net OUT_INJ6: now also J30.12
- net OUT_LS1: now also J30.19
- net OUT_LS2: now also J30.20
- net OUT_LS3: now also J30.21
- net OUT_LS4: now also J30.22
- net OUT_LS_HOT1: now also J30.23
- net OUT_LS_HOT2: now also J30.24
- net USB+: now also J30.30
- net USB-: now also J30.31
- net VBUS: now also J30.29
- net VR_DISCRETE+: now also J31.21
- net VR_DISCRETE-: now also J31.22
- net VR_MAX9924+: now also J31.23
- net VR_MAX9924-: now also J31.24
- new net 12V_HALL: F11.2, J30.6
- new net EGT2+: J33.1 (Pin_1)
- new net EGT2-: J33.2 (Pin_2)
- new net EGT3+: J34.1 (Pin_1)
- new net EGT3-: J34.2 (Pin_2)
- new net EGT4+: J35.1 (Pin_1)
- new net EGT4-: J35.2 (Pin_2)
- new net WBO2_Heater: J30.28, M8.E5 (LSU_Htr)
- new net WBO2_Ip: J31.31, M8.E3 (LSU_Ip)
- new net WBO2_Rtrim: J31.34, M8.E4 (LSU_Rtrim)
- new net WBO2_SEL2: M8.J2 (SEL2), M8.J_VCC2 (PULL_UP2)
- new net WBO2_Un: J31.33, M8.E1 (LSU_Un)
- new net WBO2_Vm: J31.32, M8.E2 (LSU_Vm)
- no-connect marks 34 -> 44
Other:
- removed sheet DC Driver 1
- removed sheet DC Driver 2
- added sheet EGT2 (egt.kicad_sch)
- added sheet EGT3 (egt.kicad_sch)
- added sheet EGT4 (egt.kicad_sch)
- note added: "WBO2: SEL1 floating + SEL2 high = HW index 5 -> Lambda 2 (WBO1: SEL1 low, SEL2 floating = HW index 1)"
- note added: "uaEFI moto: Superseal 1.0 34-pin, A = TE 6437288-1 (keying 1), B = TE 6437288-2 (keying 2)"

Commit message: uaefi-moto schematic: tidy new area [skip ci]
Co-Authored-By: Claude Opus 5.5 <noreply@anthropic.com>
Other:
- note added: "uaEFI moto: J30 = TE 6437288-1 (A), J31 = TE 6437288-2 (B)"
- note removed: "uaEFI moto: Superseal 1.0 34-pin, A = TE 6437288-1 (keying 1), B = TE 6437288-2 (keying 2)"
Changed lines of the file:
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@@
 		)
 	)
-	(text "uaEFI moto: Superseal 1.0 34-pin, A = TE 6437288-1 (keying 1), B = TE 6437288-2 (keying 2)"
+	(text "uaEFI moto: J30 = TE 6437288-1 (A), J31 = TE 6437288-2 (B)"
 		(exclude_from_sim no)
 		(at 310.04 20 0)
@@
 	(symbol
 		(lib_id "hellen-one-wbo-0.6:Module-wbo-0.6")
-		(at 345.44 190.5 0)
+		(at 370.84 190.5 0)
 		(unit 1)
 		(exclude_from_sim no)
@@
 		(dnp no)
 		(property "Reference" "M8"
-			(at 345.44 186.69 0)
+			(at 370.84 186.69 0)
 			(effects
 				(font
@@
 		)
 		(property "Value" "Module-wbo-0.6"
-			(at 345.44 184.15 0)
+			(at 370.84 184.15 0)
 			(effects
 				(font
@@
 		)
 		(property "Footprint" "hellen-one-wbo-0.6:wbo"
-			(at 345.44 190.5 0)
+			(at 370.84 190.5 0)
 			(effects
 				(font
@@
 		)
 		(property "Datasheet" ""
-			(at 345.44 190.5 0)
+			(at 370.84 190.5 0)
 			(effects
 				(font
@@
 		)
 		(property "Description" "second on-board wideband, HW index 5"
-			(at 345.44 190.5 0)
+			(at 370.84 190.5 0)
 			(effects
 				(font
@@
 	)
 	(label "WBO2_Un"
-		(at 386.08 208.28 0)
+		(at 411.48 208.28 0)
 		(effects
 			(font
@@
 	)
 	(label "WBO2_Vm"
-		(at 386.08 205.74 0)
+		(at 411.48 205.74 0)
 		(effects
 			(font
@@
 	)
 	(label "WBO2_Ip"
-		(at 386.08 203.2 0)
+		(at 411.48 203.2 0)
 		(effects
 			(font
@@
 	)
 	(label "WBO2_Rtrim"
-		(at 386.08 200.66 0)
+		(at 411.48 200.66 0)
 		(effects
 			(font
@@
 	)
 	(label "WBO2_Heater"
-		(at 386.08 198.12 0)
+		(at 411.48 198.12 0)
 		(effects
 			(font
@@
 	(wire
 		(pts
-			(xy 386.08 210.82) (xy 393.7 210.82)
+			(xy 411.48 210.82) (xy 419.1 210.82)
 		)
 		(stroke
@@
 	(symbol
 		(lib_id "power:GND")
-		(at 393.7 210.82 90)
+		(at 419.1 210.82 90)
 		(unit 1)
 		(exclude_from_sim no)
@@
 		(dnp no)
 		(property "Reference" "#PWR0518"
-			(at 393.7 207.01 0)
+			(at 419.1 207.01 0)
 			(effects
 				(font
@@
 		)
 		(property "Value" "GND"
-			(at 393.7 214.63 0)
+			(at 419.1 214.63 0)
 			(effects
 				(font
@@
 		)
 		(property "Footprint" ""
-			(at 393.7 210.82 0)
+			(at 419.1 210.82 0)
 			(effects
 				(font
@@
 		)
 		(property "Datasheet" ""
-			(at 393.7 210.82 0)
+			(at 419.1 210.82 0)
 			(effects
 				(font
@@
 		)
 		(property "Description" ""
-			(at 393.7 210.82 0)
+			(at 419.1 210.82 0)
 			(effects
 				(font
@@
 	)
 	(no_connect
-		(at 386.08 218.44)
+		(at 411.48 218.44)
 	)
 	(label "WBO2_SEL2"
-		(at 386.08 226.06 0)
+		(at 411.48 226.06 0)
 		(effects
 			(font
@@
 	)
 	(no_connect
-		(at 386.08 220.98)
+		(at 411.48 220.98)
 	)
 	(no_connect
-		(at 386.08 228.6)
+		(at 411.48 228.6)
 	)
 	(no_connect
-		(at 386.08 215.9)
+		(at 411.48 215.9)
 	)
 	(label "WBO2_SEL2"
-		(at 386.08 223.52 0)
+		(at 411.48 223.52 0)
 		(effects
 			(font
@@
 	(wire
 		(pts
-			(xy 386.08 193.04) (xy 393.7 193.04)
+			(xy 411.48 193.04) (xy 419.1 193.04)
 		)
 		(stroke
@@
 	(symbol
 		(lib_id "power:+5VA")
-		(at 393.7 193.04 270)
+		(at 419.1 193.04 270)
 		(unit 1)
 		(exclude_from_sim no)
@@
 		(dnp no)
 		(property "Reference" "#PWR0519"
-			(at 393.7 189.23 0)
+			(at 419.1 189.23 0)
 			(effects
 				(font
@@
 		)
 		(property "Value" "+5VA"
-			(at 393.7 196.85 0)
+			(at 419.1 196.85 0)
 			(effects
 				(font
@@
 		)
 		(property "Footprint" ""
-			(at 393.7 193.04 0)
+			(at 419.1 193.04 0)
 			(effects
 				(font
@@
 		)
 		(property "Datasheet" ""
-			(at 393.7 193.04 0)
+			(at 419.1 193.04 0)
 			(effects
 				(font
@@
 		)
 		(property "Description" ""
-			(at 393.7 193.04 0)
+			(at 419.1 193.04 0)
 			(effects
 				(font
@@
 	)
 	(no_connect
-		(at 337.82 193.04)
+		(at 363.22 193.04)
 	)
 	(label "CAN-"
-		(at 337.82 195.58 180)
+		(at 363.22 195.58 180)
 		(effects
 			(font
@@
 	)
 	(label "CAN+"
-		(at 337.82 198.12 180)
+		(at 363.22 198.12 180)
 		(effects
 			(font
@@
 	)
 	(no_connect
-		(at 337.82 210.82)
+		(at 363.22 210.82)
 	)
 	(no_connect
-		(at 337.82 208.28)
+		(at 363.22 208.28)
 	)
 	(no_connect
-		(at 337.82 205.74)
+		(at 363.22 205.74)
 	)
 	(no_connect
-		(at 337.82 203.2)
+		(at 363.22 203.2)
 	)
 	(no_connect
-		(at 337.82 215.9)
+		(at 363.22 215.9)
 	)
 	(text "WBO2: SEL1 floating + SEL2 high = HW index 5 -> Lambda 2 (WBO1: SEL1 low, SEL2 floating = HW index 1)"
 		(exclude_from_sim no)
-		(at 330.44 182.5 0)
+		(at 350.84 178.5 0)
 		(effects
 			(font

Commit message: uaefi-moto: new A/B split from wiring spreadsheet [skip ci]
- A = base harness (INJ/IGN/GPPWM 1-2, TPS1, CLT, IAT, crank hall, WBO1, USB, CAN, relay 1, knock)
- B = extension (INJ/IGN/GPPWM 3-4, WBO2, VR, cam hall, wheel sensors, analog, relay 2)
- INJ/IGN 5-6 not on connectors, IGN6 sheet output no-connect
- wheel sensor 2 on IN_BUTTON2: R39 4.7k populated, R36 DNP
- moto/uaefi-moto-pinout.xlsx is the source of truth for the pinout
- ERC 0 errors, netlist verified against original and against spreadsheet

Co-Authored-By: Claude Opus 5.5 <noreply@anthropic.com>
Parts:
- R38: now not fitted
- R39: value DNP -> 4.7k; LCSC (none) -> C17673
Connections:
- net OUT_IGN6 is gone; now on net IN_CLT: J30.18
- net +12V_RAW: now also J30.21, J31.29; no longer J30.25, J30.27
- net +5VP: now also J30.4, J30.5; no longer J31.1
- net 12V_HALL: now also J30.3, J31.1; no longer J30.6
- net 1_WBO_Ip: now also J30.23; no longer J31.27
- net 2_WBO_Vm: now also J30.24; no longer J31.28
- net 3_WBO_Heater: now also J30.22; no longer J30.26
- net 5_WBO_Rtrim: now also J30.26; no longer J31.30
- net 6_WBO_Un: now also J30.25; no longer J31.29
- net CAN+: now also J30.31; no longer J30.33
- net CAN-: now also J30.32; no longer J30.34
- net GND: now also J30.10, J30.30, J30.8, J30.9, J31.27, J31.4; no longer J30.3, J30.32, J30.4, J30.5, J31.25
- net GNDA: now also J30.6, J30.7; no longer J31.4, J31.5
- net IN_AUX1: now also J31.15; no longer J31.11
- net IN_AUX2: now also J31.16; no longer J31.12
- net IN_AUX3: now also J31.11; no longer J31.15
- net IN_BUTTON1: now also J31.22; no longer J31.20
- net IN_BUTTON2: now also J31.28
- net IN_CLT: no longer J31.8
- net IN_FLEX: now also J31.21; no longer J31.19
- net IN_HALL1: now also J30.20; no longer J31.16
- net IN_HALL2: now also J31.19; no longer J31.17
- net IN_HALL3: now also J31.20; no longer J31.18
- net IN_IAT: now also J30.19; no longer J31.9
- net IN_KNOCK_RAW: now also J30.34; no longer J31.26
- net IN_MAP: now also J31.14; no longer J31.10
- net IN_PPS1: now also J31.17; no longer J31.13
- net IN_PPS2: now also J31.18; no longer J31.14
- net IN_TPS1: now also J30.17; no longer J31.6
- net IN_TPS2: now also J31.13; no longer J31.7
- net OUT_IGN3: now also J31.7; no longer J30.15
- net OUT_IGN4: now also J31.8; no longer J30.16
- net OUT_IGN5: no longer J30.17
- net OUT_INJ1: now also J30.11; no longer J30.7
- net OUT_INJ2: now also J30.12; no longer J30.8
- net OUT_INJ3: now also J31.5; no longer J30.9
- net OUT_INJ4: now also J31.6; no longer J30.10
- net OUT_INJ5: no longer J30.11
- net OUT_INJ6: no longer J30.12
- net OUT_LS1: now also J30.15; no longer J30.19
- net OUT_LS2: now also J30.16; no longer J30.20
- net OUT_LS3: now also J31.9; no longer J30.21
- net OUT_LS4: now also J31.10; no longer J30.22
- net OUT_LS_HOT1: now also J30.33; no longer J30.23
- net OUT_LS_HOT2: now also J31.12; no longer J30.24
- net USB+: now also J30.28; no longer J30.30
- net USB-: now also J30.29; no longer J30.31
- net VBUS: now also J30.27; no longer J30.29
- net VR_DISCRETE+: now also J31.23; no longer J31.21
- net VR_DISCRETE-: now also J31.24; no longer J31.22
- net VR_MAX9924+: now also J31.25; no longer J31.23
- net VR_MAX9924-: now also J31.26; no longer J31.24
- net WBO2_Heater: now also J31.30; no longer J30.28
- no-connect marks 44 -> 45

Commit message: uaefi-moto: PCB prepared for routing, bluetooth fix caps [skip ci]
Schematic:
- breakout pin headers J1, J11-J24 removed (never populated)
- C40 47uF on +5V and C41 470uF on +3.3VA for the JDY-33 power-up issue
- ERC 0 errors, no existing net changed, connector pins match spreadsheet

PCB:
- old Mini-Fit connectors, DC drivers, F3/F4, breakout headers and the
  routes that only led to them removed
- board enlarged to 145 x 110 mm (right: EGT/M8, top: Superseal pin depth)
- J30/J31, F11, M8, J32-J35, four MAX31855 groups, C40/C41 pre-placed
- DRC: 0 errors except library courtyard of the Superseal footprint,
  schematic parity 0, 138 unconnected items left to route

Co-Authored-By: Claude Opus 5.5 <noreply@anthropic.com>
Parts:
- removed J1, J11, J12, J13, J14, J15, J16, J17, J18, J19, J20, J21, J22, J24: Conn_02x02_Odd_Even, Connector_PinSocket_2.54mm:PinSocket_2x02_P2.54mm_Vertical, symbol Connector_Generic:Conn_02x02_Odd_Even
- added C40: 47uF 16V, Capacitor_SMD:CP_Elec_6.3x5.4, symbol Device:C_Polarized
- added C41: 470uF 6.3V, Capacitor_SMD:CP_Elec_8x10, symbol Device:C_Polarized
Connections:
- net +3.3VA: now also C41.1
- net +5V: now also C40.1
- net GND: now also C40.2, C41.2
Other:
- note added: "Bluetooth U5 (JDY-33) power-up fix, see uaEFI README: bulk caps on +5V and +3.3VA"
